Commit message: Lots of little changes.  TCP

File: operation_description/urdf/iiwa.urdf.xacro (robot description, xacro)
@@ -11,3 +11,21 @@
     <origin xyz="$(arg origin_xyz)" rpy="$(arg origin_rpy)" />
   </xacro:iiwa7>
+  <link name="grip_link">
+    <visual>
+      <geometry>
+        <mesh filename="package://operation_description/meshes/HandESmall.dae" />
+      </geometry>
+    </visual>
+  </link>
+  <joint name="grip_joint" type="fixed">
+    <parent link="iiwa_link_ee" />
+    <child link="grip_link" />
+    <origin xyz="0 0 0" rpy="0 0 0"/>
+  </joint>
+  <link name="tweeze_tips" />
+  <joint name="tweeze_joint" type="fixed">
+    <parent link="grip_link" />
+    <child link="tweeze_tips" />
+    <origin xyz="-0.01768 0.00131 0.20735" rpy="0 2.87979 0"/>
+  </joint>
 </robot>

Commit message: Updated description and moveit config

File: operation_description/urdf/iiwa.urdf.xacro (robot description, xacro)
@@ -11,4 +11,37 @@
     <origin xyz="$(arg origin_xyz)" rpy="$(arg origin_rpy)" />
   </xacro:iiwa7>
+  <link name="table_link">
+    <visual>
+      <geometry>
+        <mesh filename="package://operation_description/meshes/Table.dae" />
+      </geometry>
+    </visual>
+  </link>
+  <joint name="table_joint" type="fixed">
+    <parent link="world" />
+    <child link="table_link" />
+  </joint>
+  <link name="game_link">
+    <visual>
+      <geometry>
+        <mesh filename="package://operation_description/meshes/Game.dae" />
+      </geometry>
+    </visual>
+  </link>
+  <joint name="game_joint" type="fixed">
+    <parent link="world" />
+    <child link="game_link" />
+  </joint>
+  <link name="wall_link">
+    <visual>
+      <geometry>
+        <mesh filename="package://operation_description/meshes/Wall.dae" />
+      </geometry>
+    </visual>
+  </link>
+  <joint name="wall_joint" type="fixed">
+    <parent link="world" />
+    <child link="wall_link" />
+  </joint>
   <link name="grip_link">
     <visual>
